File: ArduinoShield.kicad_pcb (KiCad board)
At the start: 2 copper layers, 53.3 x 55.9 mm, 364 parts, among them J1 Voltage, J10 Hole, J100 Hole, J101 Hole, J102 Hole, J103 Hole, J104 Hole, J105 Hole, J106 Hole, J107 Hole, J108 Hole, J109 Hole, J11 Hole, J110 Hole, J111 Hole, J112 Hole, J113 Hole, J114 Hole, J115 Hole, J116 Hole, J117 Hole, J118 Hole, J119 Hole, J12 Hole, J120 Hole, J121 Hole, J122 Hole, J123 Hole, J124 Hole, J125 Hole, J126 Hole, J127 Hole, J128 Hole, J129 Hole, J13 Hole, J130 Hole, J131 Hole, J132 Hole, J133 Hole, J134 Hole, J135 Hole, J136 Hole, J137 Hole, J138 Hole, J139 Hole, J14 Hole, J140 Hole, J141 Hole, J142 Hole, J143 Hole, J144 Hole, J145 Hole, J146 Hole, J147 Hole, J148 Hole, J149 Hole, J15 Hole, J150 Hole, J151 Hole, J152 Hole, J153 Hole, J154 Hole, J155 Hole, J156 Hole, J157 Hole, J158 Hole, J159 Hole, J16 Hole, J160 Hole, J161 Hole, J162 Hole, J163 Hole, J164 Hole, J165 Hole, J166 Hole, J167 Hole, J168 Hole, J169 Hole, J17 Hole, J170 Hole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

Commit message: Version 2
Parts:
- removed J147, J148, J161, J162, J163, J164, J165, J166, J181, J182, J183, J184, J197, J198, J211, J212, J213, J214, J227, J228, J229, J230, J255, J256, J257, J258, J78, J79, J80, J81, J82, J83, J84, J85, J86: Hole, Lib_Custom:BasicHole
- removed the J64 at (114.3, 73.7)
- removed the J65 at (114.3, 78.7)
- removed the J66 at (111.8, 81.3)
- removed the J67 at (109.2, 83.8)
- removed the J68 at (114.3, 86.4)
- removed the J69 at (109.2, 88.9)
- removed the J70 at (111.8, 91.4)
- removed the J71 at (142.2, 50.8)
- removed the J72 at (144.8, 53.3)
- removed the J73 at (142.2, 55.9)
- removed the J74 at (144.8, 58.4)
- removed the J75 at (142.2, 61.0)
- removed the J77 at (142.2, 66.0)
- added U111: Hole, Lib_Custom:BasicHole, F.Cu at (114.3, 76.2)
- added U112: Hole, Lib_Custom:BasicHole, F.Cu at (109.2, 50.8)
- added U126: Hole, Lib_Custom:BasicHole, F.Cu at (114.3, 78.7)
- added U127: Hole, Lib_Custom:BasicHole, F.Cu at (106.7, 50.8)
- added U141: Hole, Lib_Custom:BasicHole, F.Cu at (109.2, 55.9)
- added U142: Hole, Lib_Custom:BasicHole, F.Cu at (104.1, 53.3)
- added U155: Hole, Lib_Custom:BasicHole, F.Cu at (142.2, 81.3)
- added U156: Hole, Lib_Custom:BasicHole, F.Cu at (104.1, 58.4)
- added U157: Hole, Lib_Custom:BasicHole, F.Cu at (114.3, 91.4)
- added U16: Hole, Lib_Custom:BasicHole, F.Cu at (104.1, 55.9)
- added U17: Hole, Lib_Custom:BasicHole, F.Cu at (114.3, 53.3)
- added U170: Hole, Lib_Custom:BasicHole, F.Cu at (142.2, 53.3)
- added U171: Hole, Lib_Custom:BasicHole, F.Cu at (109.2, 53.3)
- added U172: Hole, Lib_Custom:BasicHole, F.Cu at (142.2, 86.4)
- added U18: Hole, Lib_Custom:BasicHole, F.Cu at (142.2, 66.0)
- added U185: Hole, Lib_Custom:BasicHole, F.Cu at (142.2, 55.9)
- added U186: Hole, Lib_Custom:BasicHole, F.Cu at (106.7, 53.3)
- added U187: Hole, Lib_Custom:BasicHole, F.Cu at (142.2, 61.0)
- added U2: Hole, Lib_Custom:BasicHole, F.Cu at (142.2, 71.1)
- added U200: Hole, Lib_Custom:BasicHole, F.Cu at (142.2, 68.6)
- added U201: Hole, Lib_Custom:BasicHole, F.Cu at (111.8, 76.2)
- added U202: Hole, Lib_Custom:BasicHole, F.Cu at (142.2, 83.8)
- added U215: Hole, Lib_Custom:BasicHole, F.Cu at (142.2, 58.4)
- added U216: Hole, Lib_Custom:BasicHole, F.Cu at (114.3, 83.8)
- added U217: Hole, Lib_Custom:BasicHole, F.Cu at (114.3, 66.0)
- added U230: Hole, Lib_Custom:BasicHole, F.Cu at (114.3, 61.0)
- added U231: Hole, Lib_Custom:BasicHole, F.Cu at (111.8, 58.4)
- added U232: Hole, Lib_Custom:BasicHole, F.Cu at (114.3, 71.1)
- added U245: Hole, Lib_Custom:BasicHole, F.Cu at (114.3, 88.9)
- added U246: Hole, Lib_Custom:BasicHole, F.Cu at (114.3, 58.4)
- added U247: Hole, Lib_Custom:BasicHole, F.Cu at (114.3, 68.6)
- added U260: Hole, Lib_Custom:BasicHole, F.Cu at (142.2, 50.8)
- added U261: Hole, Lib_Custom:BasicHole, F.Cu at (106.7, 58.4)
- added U262: Hole, Lib_Custom:BasicHole, F.Cu at (142.2, 78.7)
- added U275: Hole, Lib_Custom:BasicHole, F.Cu at (142.2, 63.5)
- added U276: Hole, Lib_Custom:BasicHole, F.Cu at (104.1, 50.8)
- added U277: Hole, Lib_Custom:BasicHole, F.Cu at (142.2, 76.2)
- added U290: Hole, Lib_Custom:BasicHole, F.Cu at (142.2, 88.9)
- added U291: Hole, Lib_Custom:BasicHole, F.Cu at (109.2, 58.4)
- added U292: Hole, Lib_Custom:BasicHole, F.Cu at (142.2, 73.7)
- added U3: Hole, Lib_Custom:BasicHole, F.Cu at (114.3, 63.5)
- added U32: Hole, Lib_Custom:BasicHole, F.Cu at (114.3, 55.9)
- added U33: Hole, Lib_Custom:BasicHole, F.Cu at (109.2, 76.2)
- added U34: Hole, Lib_Custom:BasicHole, F.Cu at (142.2, 91.4)
- added U48: Hole, Lib_Custom:BasicHole, F.Cu at (111.8, 53.3)
- added U49: Hole, Lib_Custom:BasicHole, F.Cu at (114.3, 50.8)
- added U50: Hole, Lib_Custom:BasicHole, F.Cu at (114.3, 86.4)
- added U64: Hole, Lib_Custom:BasicHole, F.Cu at (114.3, 73.7)
- added U65: Hole, Lib_Custom:BasicHole, F.Cu at (144.8, 71.1)
- added U79: Hole, Lib_Custom:BasicHole, F.Cu at (111.8, 50.8)
- added U80: Hole, Lib_Custom:BasicHole, F.Cu at (111.8, 55.9)
- added U94: Hole, Lib_Custom:BasicHole, F.Cu at (114.3, 81.3)
- added U95: Hole, Lib_Custom:BasicHole, F.Cu at (106.7, 55.9)
- moved J76 9.16 mm to (147.3, 71.1)
- moved J62 8.03 mm to (106.7, 71.1)
- moved J61 8.03 mm to (106.7, 68.6)
- moved J63 8.03 mm to (106.7, 73.7)
- moved J59 5.68 mm to (106.7, 63.5)
- moved J26 5.08 mm to (109.2, 63.5)
- moved J5 5.08 mm to (109.2, 83.8)
- moved J7 5.08 mm to (109.2, 88.9)
- moved J23 5.08 mm to (147.3, 88.9)
- moved J53 5.08 mm to (147.3, 78.7)
- moved J60 3.59 mm to (106.7, 66.0)
- moved J10 2.54 mm to (144.8, 53.3)
- moved J17 2.54 mm to (144.8, 73.7)
- moved J25 2.54 mm to (111.8, 61.0)
- moved J38 2.54 mm to (111.8, 81.3)
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- renumbered J87 to J64, J88 to J65, J89 to J66, J90 to J67, J91 to J68, J92 to J69, J93 to J70, J94 to J71, J95 to J72, J96 to J73, J97 to J74, J98 to J75, J99 to J77, J355 to U1, J106 to U10, J187 to U100, J188 to U101, J189 to U102, J190 to U103, J191 to U104, J192 to U105, J193 to U106, J194 to U107, J195 to U108, J196 to U109, J107 to U11, J362 to U110, J199 to U113, J200 to U114, J201 to U115, J202 to U116, J203 to U117, J204 to U118, J205 to U119, J108 to U12, J206 to U120, J207 to U121, J208 to U122, J209 to U123, J210 to U124, J363 to U125, J215 to U128, J216 to U129, J109 to U13, J217 to U130, J218 to U131, J219 to U132, J220 to U133, J221 to U134, J222 to U135, J223 to U136, J224 to U137, J225 to U138, J226 to U139, J110 to U14, J364 to U140, J231 to U143, J232 to U144, J233 to U145, J234 to U146, J235 to U147, J236 to U148, J237 to U149, J356 to U15, J238 to U150, J239 to U151, J240 to U152, J241 to U153, J242 to U154, J243 to U158, J244 to U159, J245 to U160, J246 to U161, J247 to U162, J248 to U163, J249 to U164, J250 to U165, J251 to U166, J252 to U167, J253 to U168, J254 to U169, J259 to U173, J260 to U174, J261 to U175, J262 to U176, J263 to U177, J264 to U178, J265 to U179, J266 to U180, J267 to U181, J268 to U182, J269 to U183, J270 to U184, J271 to U188, J272 to U189, J111 to U19, J273 to U190, J274 to U191, J275 to U192, J276 to U193, J277 to U194, J278 to U195, J279 to U196, J280 to U197, J281 to U198, J282 to U199, J112 to U20, J283 to U203, J284 to U204, J285 to U205, J286 to U206, J287 to U207, J288 to U208, J289 to U209, J113 to U21, J290 to U210, J291 to U211, J292 to U212, J293 to U213, J294 to U214, J295 to U218, J296 to U219, J114 to U22, J297 to U220, J298 to U221, J299 to U222, J300 to U223, J301 to U224, J302 to U225, J303 to U226, J304 to U227, J305 to U228, J306 to U229, J115 to U23, J307 to U233, J308 to U234, J309 to U235, J310 to U236, J311 to U237, J312 to U238, J313 to U239, J116 to U24, J314 to U240, J315 to U241, J316 to U242, J317 to U243, J318 to U244, J319 to U248, J320 to U249, J117 to U25, J321 to U250, J322 to U251, J323 to U252, J324 to U253, J325 to U254, J326 to U255, J327 to U256, J328 to U257, J329 to U258, J330 to U259, J118 to U26, J331 to U263, J332 to U264, J333 to U265, J334 to U266, J335 to U267, J336 to U268, J337 to U269, J119 to U27, J338 to U270, J339 to U271, J340 to U272, J341 to U273, J342 to U274, J343 to U278, J344 to U279, J120 to U28, J345 to U280, J346 to U281, J347 to U282, J348 to U283, J349 to U284, J350 to U285, J351 to U286, J352 to U287, J353 to U288, J354 to U289, J121 to U29, J122 to U30, J357 to U31, J123 to U35, J124 to U36, J125 to U37, J126 to U38, J127 to U39, J100 to U4, J128 to U40, J129 to U41, J130 to U42, J131 to U43, J132 to U44, J133 to U45, J134 to U46, J358 to U47, J101 to U5, J135 to U51, J136 to U52, J137 to U53, J138 to U54, J139 to U55, J140 to U56, J141 to U57, J142 to U58, J143 to U59, J102 to U6, J144 to U60, J145 to U61, J146 to U62, J359 to U63, J149 to U66, J150 to U67, J151 to U68, J152 to U69, J103 to U7, J153 to U70, J154 to U71, J155 to U72, J156 to U73, J157 to U74, J158 to U75, J159 to U76, J160 to U77, J360 to U78, J104 to U8, J167 to U81, J168 to U82, J169 to U83, J170 to U84, J171 to U85, J172 to U86, J173 to U87, J174 to U88, J175 to U89, J105 to U9, J176 to U90, J177 to U91, J178 to U92, J361 to U93, J179 to U96, J180 to U97, J185 to U98, J186 to U99
Connections:
- J59 pad 1: RST -> 3v3
- J60 pad 1: 3v3 -> 5v
- J61 pad 1: 5v -> GND
- J62 pad 1: GND -> GND2
- J63 pad 1: GND2 -> VIN
- J64 pad 1: Net-(J87-Pad1) -> unconnected-(J64-Pad1)
- J65 pad 1: Net-(J88-Pad1) -> unconnected-(J65-Pad1)
- J66 pad 1: Net-(J89-Pad1) -> unconnected-(J66-Pad1)
- J67 pad 1: Net-(J90-Pad1) -> unconnected-(J67-Pad1)
- J68 pad 1: Net-(J91-Pad1) -> unconnected-(J68-Pad1)
- J69 pad 1: Net-(J92-Pad1) -> unconnected-(J69-Pad1)
- J70 pad 1: Net-(J93-Pad1) -> unconnected-(J70-Pad1)
- J71 pad 1: Net-(J94-Pad1) -> unconnected-(J71-Pad1)
- J72 pad 1: Net-(J95-Pad1) -> unconnected-(J72-Pad1)
- J73 pad 1: Net-(J96-Pad1) -> unconnected-(J73-Pad1)
- J74 pad 1: Net-(J97-Pad1) -> unconnected-(J74-Pad1)
- J75 pad 1: Net-(J98-Pad1) -> unconnected-(J75-Pad1)
- J76 pad 1: 10 -> unconnected-(J76-Pad1)
- J77 pad 1: Net-(J99-Pad1) -> unconnected-(J77-Pad1)
- U1 pad 1: Net-(J355-Pad1) -> unconnected-(U1-Pad1)
- U10 pad 1: Net-(J106-Pad1) -> unconnected-(U10-Pad1)
- U100 pad 1: Net-(J187-Pad1) -> unconnected-(U100-Pad1)
- U101 pad 1: Net-(J188-Pad1) -> unconnected-(U101-Pad1)
- U102 pad 1: Net-(J189-Pad1) -> unconnected-(U102-Pad1)
- U103 pad 1: Net-(J190-Pad1) -> unconnected-(U103-Pad1)
- U104 pad 1: Net-(J191-Pad1) -> unconnected-(U104-Pad1)
- U105 pad 1: Net-(J192-Pad1) -> unconnected-(U105-Pad1)
- U106 pad 1: Net-(J193-Pad1) -> unconnected-(U106-Pad1)
- U107 pad 1: Net-(J194-Pad1) -> unconnected-(U107-Pad1)
- U108 pad 1: Net-(J195-Pad1) -> unconnected-(U108-Pad1)
- U109 pad 1: Net-(J196-Pad1) -> unconnected-(U109-Pad1)
- U11 pad 1: Net-(J107-Pad1) -> unconnected-(U11-Pad1)
- U110 pad 1: Net-(J362-Pad1) -> unconnected-(U110-Pad1)
- U113 pad 1: Net-(J199-Pad1) -> unconnected-(U113-Pad1)
- U114 pad 1: Net-(J200-Pad1) -> unconnected-(U114-Pad1)
- U115 pad 1: Net-(J201-Pad1) -> unconnected-(U115-Pad1)
- U116 pad 1: Net-(J202-Pad1) -> unconnected-(U116-Pad1)
- U117 pad 1: Net-(J203-Pad1) -> unconnected-(U117-Pad1)
- U118 pad 1: Net-(J204-Pad1) -> unconnected-(U118-Pad1)
- U119 pad 1: Net-(J205-Pad1) -> unconnected-(U119-Pad1)
- U12 pad 1: Net-(J108-Pad1) -> unconnected-(U12-Pad1)
- U120 pad 1: Net-(J206-Pad1) -> unconnected-(U120-Pad1)
- U121 pad 1: Net-(J207-Pad1) -> unconnected-(U121-Pad1)
- U122 pad 1: Net-(J208-Pad1) -> unconnected-(U122-Pad1)
- U123 pad 1: Net-(J209-Pad1) -> unconnected-(U123-Pad1)
- U124 pad 1: Net-(J210-Pad1) -> unconnected-(U124-Pad1)
- U125 pad 1: Net-(J363-Pad1) -> unconnected-(U125-Pad1)
- U128 pad 1: Net-(J215-Pad1) -> unconnected-(U128-Pad1)
- U129 pad 1: Net-(J216-Pad1) -> unconnected-(U129-Pad1)
- U13 pad 1: Net-(J109-Pad1) -> unconnected-(U13-Pad1)
- U130 pad 1: Net-(J217-Pad1) -> unconnected-(U130-Pad1)
- U131 pad 1: Net-(J218-Pad1) -> unconnected-(U131-Pad1)
- U132 pad 1: Net-(J219-Pad1) -> unconnected-(U132-Pad1)
- U133 pad 1: Net-(J220-Pad1) -> unconnected-(U133-Pad1)
- U134 pad 1: Net-(J221-Pad1) -> unconnected-(U134-Pad1)
- U135 pad 1: Net-(J222-Pad1) -> unconnected-(U135-Pad1)
- U136 pad 1: Net-(J223-Pad1) -> unconnected-(U136-Pad1)
- U137 pad 1: Net-(J224-Pad1) -> unconnected-(U137-Pad1)
- U138 pad 1: Net-(J225-Pad1) -> unconnected-(U138-Pad1)
- U139 pad 1: Net-(J226-Pad1) -> unconnected-(U139-Pad1)
- U14 pad 1: Net-(J110-Pad1) -> unconnected-(U14-Pad1)
- U140 pad 1: Net-(J364-Pad1) -> unconnected-(U140-Pad1)
- U143 pad 1: Net-(J231-Pad1) -> unconnected-(U143-Pad1)
- U144 pad 1: Net-(J232-Pad1) -> unconnected-(U144-Pad1)
- U145 pad 1: Net-(J233-Pad1) -> unconnected-(U145-Pad1)
- U146 pad 1: Net-(J234-Pad1) -> unconnected-(U146-Pad1)
- U147 pad 1: Net-(J235-Pad1) -> unconnected-(U147-Pad1)
- U148 pad 1: Net-(J236-Pad1) -> unconnected-(U148-Pad1)
- U149 pad 1: Net-(J237-Pad1) -> unconnected-(U149-Pad1)
- U15 pad 1: Net-(J356-Pad1) -> unconnected-(U15-Pad1)
- U150 pad 1: Net-(J238-Pad1) -> unconnected-(U150-Pad1)
- U151 pad 1: Net-(J239-Pad1) -> unconnected-(U151-Pad1)
- U152 pad 1: Net-(J240-Pad1) -> unconnected-(U152-Pad1)
- U153 pad 1: Net-(J241-Pad1) -> unconnected-(U153-Pad1)
- U154 pad 1: Net-(J242-Pad1) -> unconnected-(U154-Pad1)
- U158 pad 1: Net-(J243-Pad1) -> unconnected-(U158-Pad1)
- U159 pad 1: Net-(J244-Pad1) -> unconnected-(U159-Pad1)
- U160 pad 1: Net-(J245-Pad1) -> unconnected-(U160-Pad1)
- U161 pad 1: Net-(J246-Pad1) -> unconnected-(U161-Pad1)
- U162 pad 1: Net-(J247-Pad1) -> unconnected-(U162-Pad1)
- U163 pad 1: Net-(J248-Pad1) -> unconnected-(U163-Pad1)
- U164 pad 1: Net-(J249-Pad1) -> unconnected-(U164-Pad1)
- U165 pad 1: Net-(J250-Pad1) -> unconnected-(U165-Pad1)
- U166 pad 1: Net-(J251-Pad1) -> unconnected-(U166-Pad1)
- U167 pad 1: Net-(J252-Pad1) -> unconnected-(U167-Pad1)
- U168 pad 1: Net-(J253-Pad1) -> unconnected-(U168-Pad1)
- U169 pad 1: Net-(J254-Pad1) -> unconnected-(U169-Pad1)
- U173 pad 1: Net-(J259-Pad1) -> unconnected-(U173-Pad1)
- U174 pad 1: Net-(J260-Pad1) -> unconnected-(U174-Pad1)
- U175 pad 1: Net-(J261-Pad1) -> unconnected-(U175-Pad1)
- U176 pad 1: Net-(J262-Pad1) -> unconnected-(U176-Pad1)
- U177 pad 1: Net-(J263-Pad1) -> unconnected-(U177-Pad1)
- U178 pad 1: Net-(J264-Pad1) -> unconnected-(U178-Pad1)
- U179 pad 1: Net-(J265-Pad1) -> unconnected-(U179-Pad1)
- U180 pad 1: Net-(J266-Pad1) -> unconnected-(U180-Pad1)
- U181 pad 1: Net-(J267-Pad1) -> unconnected-(U181-Pad1)
- U182 pad 1: Net-(J268-Pad1) -> unconnected-(U182-Pad1)
- U183 pad 1: Net-(J269-Pad1) -> unconnected-(U183-Pad1)
- U184 pad 1: Net-(J270-Pad1) -> unconnected-(U184-Pad1)
- U188 pad 1: Net-(J271-Pad1) -> unconnected-(U188-Pad1)
- U189 pad 1: Net-(J272-Pad1) -> unconnected-(U189-Pad1)
- U19 pad 1: Net-(J111-Pad1) -> unconnected-(U19-Pad1)
- U190 pad 1: Net-(J273-Pad1) -> unconnected-(U190-Pad1)
- U191 pad 1: Net-(J274-Pad1) -> unconnected-(U191-Pad1)
- U192 pad 1: Net-(J275-Pad1) -> unconnected-(U192-Pad1)
- U193 pad 1: Net-(J276-Pad1) -> unconnected-(U193-Pad1)
- U194 pad 1: Net-(J277-Pad1) -> unconnected-(U194-Pad1)
- U195 pad 1: Net-(J278-Pad1) -> unconnected-(U195-Pad1)
- U196 pad 1: Net-(J279-Pad1) -> unconnected-(U196-Pad1)
- U197 pad 1: Net-(J280-Pad1) -> unconnected-(U197-Pad1)
- U198 pad 1: Net-(J281-Pad1) -> unconnected-(U198-Pad1)
- U199 pad 1: Net-(J282-Pad1) -> unconnected-(U199-Pad1)
- U20 pad 1: Net-(J112-Pad1) -> unconnected-(U20-Pad1)
- U203 pad 1: Net-(J283-Pad1) -> unconnected-(U203-Pad1)
- U204 pad 1: Net-(J284-Pad1) -> unconnected-(U204-Pad1)
- U205 pad 1: Net-(J285-Pad1) -> unconnected-(U205-Pad1)
- U206 pad 1: Net-(J286-Pad1) -> unconnected-(U206-Pad1)
- U207 pad 1: Net-(J287-Pad1) -> unconnected-(U207-Pad1)
- U208 pad 1: Net-(J288-Pad1) -> unconnected-(U208-Pad1)
- U209 pad 1: Net-(J289-Pad1) -> unconnected-(U209-Pad1)
- U21 pad 1: Net-(J113-Pad1) -> unconnected-(U21-Pad1)
- U210 pad 1: Net-(J290-Pad1) -> unconnected-(U210-Pad1)
- U211 pad 1: Net-(J291-Pad1) -> unconnected-(U211-Pad1)
- U212 pad 1: Net-(J292-Pad1) -> unconnected-(U212-Pad1)
- U213 pad 1: Net-(J293-Pad1) -> unconnected-(U213-Pad1)
- U214 pad 1: Net-(J294-Pad1) -> unconnected-(U214-Pad1)
- U218 pad 1: Net-(J295-Pad1) -> unconnected-(U218-Pad1)
- U219 pad 1: Net-(J296-Pad1) -> unconnected-(U219-Pad1)
- U22 pad 1: Net-(J114-Pad1) -> unconnected-(U22-Pad1)
- U220 pad 1: Net-(J297-Pad1) -> unconnected-(U220-Pad1)
- U221 pad 1: Net-(J298-Pad1) -> unconnected-(U221-Pad1)
- U222 pad 1: Net-(J299-Pad1) -> unconnected-(U222-Pad1)
- U223 pad 1: Net-(J300-Pad1) -> unconnected-(U223-Pad1)
- U224 pad 1: Net-(J301-Pad1) -> unconnected-(U224-Pad1)
- U225 pad 1: Net-(J302-Pad1) -> unconnected-(U225-Pad1)
- U226 pad 1: Net-(J303-Pad1) -> unconnected-(U226-Pad1)
- U227 pad 1: Net-(J304-Pad1) -> unconnected-(U227-Pad1)
- U228 pad 1: Net-(J305-Pad1) -> unconnected-(U228-Pad1)
- U229 pad 1: Net-(J306-Pad1) -> unconnected-(U229-Pad1)
- U23 pad 1: Net-(J115-Pad1) -> unconnected-(U23-Pad1)
- U233 pad 1: Net-(J307-Pad1) -> unconnected-(U233-Pad1)
- U234 pad 1: Net-(J308-Pad1) -> unconnected-(U234-Pad1)
- U235 pad 1: Net-(J309-Pad1) -> unconnected-(U235-Pad1)
- U236 pad 1: Net-(J310-Pad1) -> unconnected-(U236-Pad1)
- U237 pad 1: Net-(J311-Pad1) -> unconnected-(U237-Pad1)
- U238 pad 1: Net-(J312-Pad1) -> unconnected-(U238-Pad1)
- U239 pad 1: Net-(J313-Pad1) -> unconnected-(U239-Pad1)
- U24 pad 1: Net-(J116-Pad1) -> unconnected-(U24-Pad1)
- U240 pad 1: Net-(J314-Pad1) -> unconnected-(U240-Pad1)
- U241 pad 1: Net-(J315-Pad1) -> unconnected-(U241-Pad1)
- U242 pad 1: Net-(J316-Pad1) -> unconnected-(U242-Pad1)
- U243 pad 1: Net-(J317-Pad1) -> unconnected-(U243-Pad1)
- U244 pad 1: Net-(J318-Pad1) -> unconnected-(U244-Pad1)
- U248 pad 1: Net-(J319-Pad1) -> unconnected-(U248-Pad1)
- U249 pad 1: Net-(J320-Pad1) -> unconnected-(U249-Pad1)
- U25 pad 1: Net-(J117-Pad1) -> unconnected-(U25-Pad1)
- U250 pad 1: Net-(J321-Pad1) -> unconnected-(U250-Pad1)
- U251 pad 1: Net-(J322-Pad1) -> unconnected-(U251-Pad1)
- U252 pad 1: Net-(J323-Pad1) -> unconnected-(U252-Pad1)
- U253 pad 1: Net-(J324-Pad1) -> unconnected-(U253-Pad1)
- U254 pad 1: Net-(J325-Pad1) -> unconnected-(U254-Pad1)
- U255 pad 1: Net-(J326-Pad1) -> unconnected-(U255-Pad1)
- U256 pad 1: Net-(J327-Pad1) -> unconnected-(U256-Pad1)
- U257 pad 1: Net-(J328-Pad1) -> unconnected-(U257-Pad1)
- U258 pad 1: Net-(J329-Pad1) -> unconnected-(U258-Pad1)
- U259 pad 1: Net-(J330-Pad1) -> unconnected-(U259-Pad1)
- U26 pad 1: Net-(J118-Pad1) -> unconnected-(U26-Pad1)
- U263 pad 1: Net-(J331-Pad1) -> unconnected-(U263-Pad1)
- U264 pad 1: Net-(J332-Pad1) -> unconnected-(U264-Pad1)
- U265 pad 1: Net-(J333-Pad1) -> unconnected-(U265-Pad1)
- U266 pad 1: Net-(J334-Pad1) -> unconnected-(U266-Pad1)
- U267 pad 1: Net-(J335-Pad1) -> unconnected-(U267-Pad1)
- U268 pad 1: Net-(J336-Pad1) -> unconnected-(U268-Pad1)
- U269 pad 1: Net-(J337-Pad1) -> unconnected-(U269-Pad1)
- U27 pad 1: Net-(J119-Pad1) -> unconnected-(U27-Pad1)
- U270 pad 1: Net-(J338-Pad1) -> unconnected-(U270-Pad1)
- U271 pad 1: Net-(J339-Pad1) -> unconnected-(U271-Pad1)
- U272 pad 1: Net-(J340-Pad1) -> unconnected-(U272-Pad1)
- U273 pad 1: Net-(J341-Pad1) -> unconnected-(U273-Pad1)
- U274 pad 1: Net-(J342-Pad1) -> unconnected-(U274-Pad1)
- U278 pad 1: Net-(J343-Pad1) -> unconnected-(U278-Pad1)
- U279 pad 1: Net-(J344-Pad1) -> unconnected-(U279-Pad1)
- U28 pad 1: Net-(J120-Pad1) -> unconnected-(U28-Pad1)
- U280 pad 1: Net-(J345-Pad1) -> unconnected-(U280-Pad1)
- U281 pad 1: Net-(J346-Pad1) -> unconnected-(U281-Pad1)
- U282 pad 1: Net-(J347-Pad1) -> unconnected-(U282-Pad1)
- U283 pad 1: Net-(J348-Pad1) -> unconnected-(U283-Pad1)
- U284 pad 1: Net-(J349-Pad1) -> unconnected-(U284-Pad1)
- U285 pad 1: Net-(J350-Pad1) -> unconnected-(U285-Pad1)
- U286 pad 1: Net-(J351-Pad1) -> unconnected-(U286-Pad1)
- U287 pad 1: Net-(J352-Pad1) -> unconnected-(U287-Pad1)
- U288 pad 1: Net-(J353-Pad1) -> unconnected-(U288-Pad1)
- U289 pad 1: Net-(J354-Pad1) -> unconnected-(U289-Pad1)
- U29 pad 1: Net-(J121-Pad1) -> unconnected-(U29-Pad1)
- U30 pad 1: Net-(J122-Pad1) -> unconnected-(U30-Pad1)
- U31 pad 1: Net-(J357-Pad1) -> unconnected-(U31-Pad1)
- U35 pad 1: Net-(J123-Pad1) -> unconnected-(U35-Pad1)
- U36 pad 1: Net-(J124-Pad1) -> unconnected-(U36-Pad1)
- U37 pad 1: Net-(J125-Pad1) -> unconnected-(U37-Pad1)
- U38 pad 1: Net-(J126-Pad1) -> unconnected-(U38-Pad1)
- U39 pad 1: Net-(J127-Pad1) -> unconnected-(U39-Pad1)
- U4 pad 1: Net-(J100-Pad1) -> unconnected-(U4-Pad1)
- U40 pad 1: Net-(J128-Pad1) -> unconnected-(U40-Pad1)
- U41 pad 1: Net-(J129-Pad1) -> unconnected-(U41-Pad1)
- U42 pad 1: Net-(J130-Pad1) -> unconnected-(U42-Pad1)
- U43 pad 1: Net-(J131-Pad1) -> unconnected-(U43-Pad1)
- U44 pad 1: Net-(J132-Pad1) -> unconnected-(U44-Pad1)
- U45 pad 1: Net-(J133-Pad1) -> unconnected-(U45-Pad1)
- U46 pad 1: Net-(J134-Pad1) -> unconnected-(U46-Pad1)
- U47 pad 1: Net-(J358-Pad1) -> unconnected-(U47-Pad1)
- U5 pad 1: Net-(J101-Pad1) -> unconnected-(U5-Pad1)
- U51 pad 1: Net-(J135-Pad1) -> unconnected-(U51-Pad1)
- U52 pad 1: Net-(J136-Pad1) -> unconnected-(U52-Pad1)
- U53 pad 1: Net-(J137-Pad1) -> unconnected-(U53-Pad1)
- U54 pad 1: Net-(J138-Pad1) -> unconnected-(U54-Pad1)
- U55 pad 1: Net-(J139-Pad1) -> unconnected-(U55-Pad1)
- U56 pad 1: Net-(J140-Pad1) -> unconnected-(U56-Pad1)
- U57 pad 1: Net-(J141-Pad1) -> unconnected-(U57-Pad1)
- U58 pad 1: Net-(J142-Pad1) -> unconnected-(U58-Pad1)
- U59 pad 1: Net-(J143-Pad1) -> unconnected-(U59-Pad1)
- U6 pad 1: Net-(J102-Pad1) -> unconnected-(U6-Pad1)
- U60 pad 1: Net-(J144-Pad1) -> unconnected-(U60-Pad1)
- U61 pad 1: Net-(J145-Pad1) -> unconnected-(U61-Pad1)
- U62 pad 1: Net-(J146-Pad1) -> unconnected-(U62-Pad1)
- U63 pad 1: Net-(J359-Pad1) -> unconnected-(U63-Pad1)
- U66 pad 1: Net-(J149-Pad1) -> unconnected-(U66-Pad1)
- U67 pad 1: Net-(J150-Pad1) -> unconnected-(U67-Pad1)
- U68 pad 1: Net-(J151-Pad1) -> unconnected-(U68-Pad1)
- U69 pad 1: Net-(J152-Pad1) -> unconnected-(U69-Pad1)
- U7 pad 1: Net-(J103-Pad1) -> unconnected-(U7-Pad1)
- U70 pad 1: Net-(J153-Pad1) -> unconnected-(U70-Pad1)
- U71 pad 1: Net-(J154-Pad1) -> unconnected-(U71-Pad1)
- U72 pad 1: Net-(J155-Pad1) -> unconnected-(U72-Pad1)
- U73 pad 1: Net-(J156-Pad1) -> unconnected-(U73-Pad1)
- U74 pad 1: Net-(J157-Pad1) -> unconnected-(U74-Pad1)
- U75 pad 1: Net-(J158-Pad1) -> unconnected-(U75-Pad1)
- U76 pad 1: Net-(J159-Pad1) -> unconnected-(U76-Pad1)
- U77 pad 1: Net-(J160-Pad1) -> unconnected-(U77-Pad1)
- U78 pad 1: Net-(J360-Pad1) -> unconnected-(U78-Pad1)
- U8 pad 1: Net-(J104-Pad1) -> unconnected-(U8-Pad1)
- U81 pad 1: Net-(J167-Pad1) -> unconnected-(U81-Pad1)
- U82 pad 1: Net-(J168-Pad1) -> unconnected-(U82-Pad1)
- U83 pad 1: Net-(J169-Pad1) -> unconnected-(U83-Pad1)
- U84 pad 1: Net-(J170-Pad1) -> unconnected-(U84-Pad1)
- U85 pad 1: Net-(J171-Pad1) -> unconnected-(U85-Pad1)
- U86 pad 1: Net-(J172-Pad1) -> unconnected-(U86-Pad1)
- U87 pad 1: Net-(J173-Pad1) -> unconnected-(U87-Pad1)
- U88 pad 1: Net-(J174-Pad1) -> unconnected-(U88-Pad1)
- U89 pad 1: Net-(J175-Pad1) -> unconnected-(U89-Pad1)
- U9 pad 1: Net-(J105-Pad1) -> unconnected-(U9-Pad1)
- U90 pad 1: Net-(J176-Pad1) -> unconnected-(U90-Pad1)
- U91 pad 1: Net-(J177-Pad1) -> unconnected-(U91-Pad1)
- U92 pad 1: Net-(J178-Pad1) -> unconnected-(U92-Pad1)
- U93 pad 1: Net-(J361-Pad1) -> unconnected-(U93-Pad1)
- U98 pad 1: Net-(J185-Pad1) -> unconnected-(U98-Pad1)
- U99 pad 1: Net-(J186-Pad1) -> unconnected-(U99-Pad1)
Routing:
- net LBLANK5: track 20.3 -> 0.00 mm
- net LBLANK4: track 20.3 -> 0.00 mm
- net LBLANK3: track 20.3 -> 0.00 mm
- net LBLANK2: track 20.3 -> 0.00 mm
- net LBLANK: track 10.2 -> 0.00 mm
- net RBLANK: track 10.2 -> 0.00 mm
- net VIN: track 20.3 -> 15.2 mm
- net RST: track 20.3 -> 15.2 mm
- net GND2: track 20.3 -> 15.2 mm
- net GND: track 20.3 -> 15.2 mm
- net A5: track 20.3 -> 15.2 mm
- net A4: track 20.3 -> 15.2 mm
- net A3: track 20.3 -> 15.2 mm
- net A2: track 20.3 -> 15.2 mm
- net A1: track 20.3 -> 15.2 mm
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Other:
- board size 53.3 x 55.9 mm -> 53.3 x 58.4 mm
- net class Default removed
- board text added: "ADBeta"
- board text added: "Mini Protoboard Shield"
